Commit message: bucking bar bigger

File: urdf/panda/panda_arm_kdl.urdf (robot description, URDF)
Before this commit: robot panda, 11 links, 10 joints
Links:
- link panda_grasptarget: mass 0.0 -> 0.1; geometry visual box size=0.02 0.02 0.1
Joints:
- joint panda_grasptarget_hand: origin xyz=0 0 0.1334 rpy=0 0 0 -> xyz=0 0 0.1934 rpy=0 0 0

File: urdf/panda/panda_arm_rivet.urdf (robot description, URDF)
Before this commit: robot panda, 13 links, 12 joints
Links:
- link panda_grasptarget: geometry visual box size=0.02 0.02 0.1
Joints:
- joint panda_grasptarget_hand: origin xyz=0 0 0.1334 rpy=0 0 0 -> xyz=0 0 0.1934 rpy=0 0 0
